Commit message: added a laser scanner to the arm

File: youbot_common/youbot_description/urdf/sensors/hokuyo_urg04_laser.urdf.xacro (robot description, xacro)
@@ -9,5 +9,5 @@
       <axis xyz="0 1 0" />
       <insert_block name="origin" />
-      <parent link="${parent}_link"/>
+      <parent link="${parent}"/>
       <child link="${name}_link"/>
     </joint>

File: youbot_common/youbot_description/urdf/youbot_arm/arm.urdf.xacro (robot description, xacro)
@@ -4,4 +4,6 @@
         xmlns:interface="http://playerstage.sourceforge.net/gazebo/xmlschema/#interface"
         xmlns:xacro="http://ros.org/wiki/xacro">
+	<!-- sensors -->
+	<include filename="$(find youbot_description)/urdf/sensors/hokuyo_urg04_laser.urdf.xacro"/>
 	<include filename="$(find youbot_description)/urdf/youbot_arm/arm.gazebo.xacro" />
 	<include filename="$(find youbot_description)/urdf/youbot_arm/arm.transmission.xacro" />
@@ -211,4 +213,7 @@
 			</collision>
 		</link>
+		<xacro:hokuyo_urg04_laser name="${name}_laser_front" parent="${name}_link_5"  ros_topic="scan_from_arm" update_rate="10" min_angle="-2.09" max_angle="2.09" >
+     			 <origin xyz="-0.060 0 0.0038" rpy="0 -${M_PI/2.0} 0" />
+    		</xacro:hokuyo_urg04_laser>
 		<!-- extensions -->
 		<xacro:youbot_arm_gazebo name="${name}" />

File: youbot_common/youbot_description/urdf/youbot_base/base.urdf.xacro (robot description, xacro)
@@ -83,5 +83,5 @@
     		</link>
 		<!-- base laser front -->
-    		<xacro:hokuyo_urg04_laser name="${name}_laser_front" parent="${name}" ros_topic="scan_front" update_rate="10" min_angle="-2.09" max_angle="2.09" >
+    		<xacro:hokuyo_urg04_laser name="${name}_laser_front" parent="${name}_link" ros_topic="scan_front" update_rate="10" min_angle="-2.09" max_angle="2.09" >
      			 <origin xyz="0.3 0 -0.03" rpy="0 0 0" />
     		</xacro:hokuyo_urg04_laser>
